File: Kicad/Circuits-imprimés/Chenillard-32-leds/Chenillard-32-leds.kicad_pcb (KiCad board)
At the start: 2 copper layers, 140 x 140 mm, 40 parts, among them J1 Conn_01x02, J2 Conn_01x02, J3 DB25_Female_MountingHoles, J4 DB25_Female_MountingHoles, U1 NE555, U2 4081, U3 4017, U4 4017, U5 4017, U6 4017

Commit message: Update project
Update project
Parts:
- moved C6 260.8 mm to (61.0, 54.6), turned to 90 degrees
- moved D1 259.0 mm to (36.2, 113.0), turned to 90 degrees
- moved J2 258.9 mm to (36.2, 121.3), turned to 90 degrees
- moved R2 254.2 mm to (55.9, 118.1), turned to 90 degrees
- moved C5 248.9 mm to (72.4, 67.9), turned to 90 degrees
- moved C7 244.7 mm to (72.4, 54.0), turned to 90 degrees
- moved C10 241.2 mm to (72.4, 156.2), turned to 90 degrees
- moved C8 239.9 mm to (71.8, 90.2), turned to 90 degrees
- moved R4 235.8 mm to (76.2, 62.9), turned to 270 degrees
- moved C9 232.2 mm to (70.5, 121.9), turned to 90 degrees
- moved R8 230.5 mm to (92.1, 167.0)
- moved R5 227.2 mm to (80.0, 70.5), turned to 90 degrees
- moved U2 223.8 mm to (61.0, 133.3), turned to 270 degrees
- moved R7 218.3 mm to (86.4, 130.2), turned to 270 degrees
- moved D5 218.1 mm to (91.4, 96.5), turned to 270 degrees
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Connections:
- C5 pad 2: GND -> +9V
- J3 pad 11: Net-(J3-Pad10) -> Net-(J3-Pad11)
- J3 pad 12: Net-(J3-Pad10) -> Net-(J3-Pad11)
- J3 pad 13: Net-(J3-Pad10) -> Net-(J3-Pad11)
- J3 pad 20: Net-(J3-Pad20) -> Net-(J3-Pad11)
- J3 pad 21: Net-(J3-Pad21) -> Net-(J3-Pad11)
- J3 pad 22: Net-(J3-Pad10) -> Net-(J3-Pad11)
- J3 pad 23: Net-(J3-Pad10) -> Net-(J3-Pad11)
- J3 pad 24: Net-(J3-Pad10) -> Net-(J3-Pad11)
- J3 pad 25: Net-(J3-Pad10) -> Net-(J3-Pad11)
- J3 pad 9: Net-(J3-Pad10) -> Net-(J3-Pad9)
- J4 pad 11: Net-(J4-Pad10) -> Net-(J4-Pad11)
- J4 pad 12: Net-(J4-Pad10) -> Net-(J4-Pad11)
- J4 pad 13: Net-(J4-Pad10) -> Net-(J4-Pad11)
- J4 pad 20: Net-(J4-Pad20) -> Net-(J4-Pad11)
- J4 pad 21: Net-(J4-Pad21) -> Net-(J4-Pad11)
- J4 pad 22: Net-(J4-Pad10) -> Net-(J4-Pad11)
- J4 pad 23: Net-(J4-Pad10) -> Net-(J4-Pad11)
- J4 pad 24: Net-(J4-Pad10) -> Net-(J4-Pad11)
- J4 pad 25: Net-(J4-Pad10) -> Net-(J4-Pad11)
- R10 pad 2: Net-(J4-Pad10) -> Net-(J4-Pad11)
- R9 pad 2: Net-(J3-Pad10) -> Net-(J3-Pad11)
- U3 pad 1: Net-(J3-Pad3) -> Net-(J3-Pad14)
- U3 pad 10: Net-(J3-Pad15) -> Net-(J3-Pad2)
- U3 pad 2: Net-(J3-Pad1) -> Net-(J3-Pad15)
- U3 pad 4: Net-(J3-Pad14) -> Net-(J3-Pad16)
- U3 pad 5: Net-(J3-Pad16) -> Net-(J3-Pad17)
- U3 pad 6: Net-(J3-Pad4) -> Net-(J3-Pad18)
- U3 pad 7: Net-(J3-Pad2) -> Net-(J3-Pad19)
- U3 pad 9: Net-(J3-Pad17) -> Net-(J3-Pad1)
- U4 pad 1: Net-(J3-Pad7) -> Net-(J3-Pad8)
- U4 pad 10: Net-(J3-Pad19) -> Net-(J3-Pad10)
- U4 pad 2: Net-(J3-Pad5) -> Net-(J3-Pad7)
- U4 pad 4: Net-(J3-Pad18) -> Net-(J3-Pad6)
- U4 pad 5: Net-(J3-Pad20) -> Net-(J3-Pad5)
- U4 pad 6: Net-(J3-Pad8) -> Net-(J3-Pad4)
- U4 pad 7: Net-(J3-Pad6) -> Net-(J3-Pad3)
- U4 pad 9: Net-(J3-Pad21) -> Net-(J3-Pad9)
- U5 pad 1: Net-(J4-Pad3) -> Net-(J4-Pad14)
- U5 pad 10: Net-(J4-Pad15) -> Net-(J4-Pad2)
- U5 pad 2: Net-(J4-Pad1) -> Net-(J4-Pad15)
- U5 pad 4: Net-(J4-Pad14) -> Net-(J4-Pad16)
- U5 pad 5: Net-(J4-Pad16) -> Net-(J4-Pad17)
- U5 pad 6: Net-(J4-Pad4) -> Net-(J4-Pad18)
- U5 pad 7: Net-(J4-Pad2) -> Net-(J4-Pad19)
- U5 pad 9: Net-(J4-Pad17) -> Net-(J4-Pad1)
- U6 pad 1: Net-(J4-Pad20) -> Net-(J4-Pad8)
- U6 pad 10: Net-(J4-Pad7) -> Net-(J4-Pad10)
- U6 pad 2: Net-(J4-Pad18) -> Net-(J4-Pad7)
- U6 pad 3: Net-(J4-Pad5) -> (no net)
- U6 pad 5: Net-(J4-Pad8) -> Net-(J4-Pad5)
- U6 pad 6: Net-(J4-Pad21) -> Net-(J4-Pad4)
- U6 pad 7: Net-(J4-Pad19) -> Net-(J4-Pad3)
Routing:
- net GND: track 69.7 -> 588.8 mm, vias 0 -> 7
- net +9V: track 31.3 -> 428.1 mm, vias 0 -> 10
- net RAZ: track 0.00 -> 187.5 mm, vias 0 -> 5
- net Horloge: track 0.00 -> 179.7 mm, vias 0 -> 2
- net Net-(D3-Pad2): track 0.00 -> 153.2 mm, vias 0 -> 2
- net Net-(U2-Pad5): track 0.00 -> 105.4 mm
- net Net-(J4-Pad19): track 0.00 -> 96.9 mm
- net Net-(J3-Pad19): track 0.00 -> 94.6 mm
- net Net-(J4-Pad18): track 0.00 -> 88.9 mm
- net Net-(U2-Pad8): track 0.00 -> 87.4 mm, vias 0 -> 2
- net Net-(J3-Pad18): track 0.00 -> 85.9 mm
- net Net-(J4-Pad17): track 0.00 -> 80.9 mm
- net Net-(J3-Pad17): track 0.00 -> 77.8 mm
- net Net-(D7-Pad2): track 0.00 -> 75.9 mm, vias 0 -> 2
- net Net-(D5-Pad2): track 0.00 -> 75.7 mm, vias 0 -> 2
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Other:
- board size 140 x 140 mm -> 105 x 140 mm
- net class Default: clearance 0.4 -> 0.2
- rule trace_clearance: 0.4 -> 0.2
