File: Kicad/Circuits-imprimés/Chenillard-32-leds/Chenillard-32-leds.sch (KiCad schematic (older format))
At the start: 40 parts, among them J1 Conn_01x02, J2 Conn_01x02, J3 DB25_Female_MountingHoles, J4 DB25_Female_MountingHoles, U1 NE555, U2 4081, U3 4017, U4 4017, U5 4017, U6 4017

Commit message: Update project
Update project
Connections:
- net +9V: now also C5.2
- net GND: no longer C5.2
- net at J3.1: now also U3.9 (Q8); no longer U3.2 (Q1)
- net at J3.11, J3.12, J3.13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: now also J3.20 (P20), J3.21 (P21); no longer J3.10, J3.9
- net at J3.14 (P14): now also U3.1 (Q5); no longer U3.4 (Q2)
- net at J3.15 (P15): now also U3.2 (Q1); no longer U3.10 (Q4)
- net at J3.16 (P16): now also U3.4 (Q2); no longer U3.5 (Q6)
- net at J3.17 (P17): now also U3.5 (Q6); no longer U3.9 (Q8)
- net at J3.18 (P18): now also U3.6 (Q7); no longer U4.4 (Q2)
- net at U4.10 (Q4): now also J3.10; no longer J3.19 (P19)
- net at U3.7 (Q3): now also J3.19 (P19); no longer J3.2
- net at U4.5 (Q6): now also J3.5; no longer J3.20 (P20)
- net at U4.9 (Q8): now also J3.9; no longer J3.21 (P21)
- net at J3.3: now also U4.7 (Q3); no longer U3.1 (Q5)
- net at J3.4: now also U4.6 (Q7); no longer U3.6 (Q7)
- net at U4.2 (Q1): now also J3.7; no longer J3.5
- net at J3.6: now also U4.4 (Q2); no longer U4.7 (Q3)
- net at U4.1 (Q5): now also J3.8; no longer J3.7
- net at J4.1: now also U5.9 (Q8); no longer U5.2 (Q1)
- net at J4.11, J4.12, J4.13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: now also J4.20 (P20), J4.21 (P21); no longer J4.10
- net at J4.14 (P14): now also U5.1 (Q5); no longer U5.4 (Q2)
- net at J4.15 (P15): now also U5.2 (Q1); no longer U5.10 (Q4)
- net at J4.16 (P16): now also U5.4 (Q2); no longer U5.5 (Q6)
- net at J4.17 (P17): now also U5.5 (Q6); no longer U5.9 (Q8)
- net at J4.18 (P18): now also U5.6 (Q7); no longer U6.2 (Q1)
- net at J4.19 (P19): now also U5.7 (Q3); no longer U6.7 (Q3)
- net at J4.2: now also U5.10 (Q4); no longer U5.7 (Q3)
- net at U6.1 (Q5): now also J4.8; no longer J4.20 (P20)
- net at U6.6 (Q7): now also J4.4; no longer J4.21 (P21)
- net at J4.3: now also U6.7 (Q3); no longer U5.1 (Q5)
- net at J4.5: now also U6.5 (Q6); no longer U6.3 (Q0)
- net at U6.10 (Q4): now also J4.10; no longer J4.7
- new net: J3.2, U3.10 (Q4)
- new net: J4.7, U6.2 (Q1)
Other:
- moved on the sheet: C5
